Commit message: update stretch urdf to make the base move

File: src/curobo/content/assets/robot/stretch_description/stretch.urdf (robot description, URDF)
Before this commit: robot stretch_description, 44 links, 43 joints
Links:
- removed link rotation_link
- removed link translation_link
- added link base_ground
- added link base_link_x
- added link base_link_y
- added link base_link_z
Joints:
- removed joint rotation_z
- added joint base_fixed: type fixed, parent base_link_z, child base_link, origin xyz=0 0 0.1 rpy=0 0 0.0, axis 0 0 0
- added joint base_y: type prismatic, parent base_link_x, child base_link_y, origin xyz=0 0 0.0 rpy=0 0 0.0, axis 0 1 0, limit lower=-5.0 upper=5.0 effort=87 velocity=1.0
- added joint base_z: type revolute, parent base_link_y, child base_link_z, origin xyz=0 0 0.0 rpy=0 0 0.0, axis 0 0 1, limit lower=-6.0 upper=6.0 effort=87 velocity=1.50
- joint base_x: axis (none) -> 1 0 0; child rotation_link -> base_link_x; limit (none) -> lower=-5.0 upper=5.0 effort=87 velocity=1.0; origin xyz=0.0 0 0 rpy=0 0 0 -> xyz=0 0 0.0 rpy=0 0 0.0; parent translation_link -> base_ground

Commit message: remove base_y joint

File: src/curobo/content/assets/robot/stretch_description/stretch.urdf (robot description, URDF)
Before this commit: robot stretch_description, 46 links, 45 joints
Joints:
- removed joint base_y
- joint base_x: limit lower=-5.0 upper=5.0 effort=87 velocity=1.0 -> lower=-500.0 upper=500.0 effort=87 velocity=1.0
- joint base_z: parent base_link_y -> base_link_x
